Commit message: Added wheels Added wheels to the axle joints

File: src/swerve_description/urdf/parts/swerve_axle.xacro (robot description, xacro)
@@ -1,35 +1,62 @@
 <?xml version="1.0"?>
 <robot xmlns:xacro="http://www.ros.org/wiki/xacro">
-  <!-- Chassis Properties -->
-  <xacro:property name="axle_length" value="0.075" />
-  <xacro:property name="axle_height" value=".1" />
-  <xacro:property name="axle_width" value="0.075" />
-  <xacro:property name="axle_weight" value="2.45" />
-  <xacro:macro name="swerve_axle" params="prefix parent *origin">
-    <link name="${prefix}_axle_link">
-      <xacro:inertial_box mass="${axle_weight}" x="${axle_length}" y="${axle_width}" z="${axle_height}">
-        <origin xyz="0 0 0" rpy="0 0 0"/>
-      </xacro:inertial_box>
-      <visual>
-        <origin xyz="0 0 0" rpy="0 0 0"/>
-        <geometry>
-          <mesh filename="package://swerve_description/meshes/SwerveAxle.stl" scale="0.001 0.001 0.001" />
-        </geometry>
-        <material name="blue"/>
-      </visual>
-      <collision>
-        <origin xyz="0 0 0" rpy="0 0 0"/>
-        <geometry>
-            <box size="${axle_length} ${axle_width} ${axle_height}" />
-        </geometry>
-      </collision>
-    </link>
-    <joint name="${prefix}_axle_joint" type="continuous">
-        <parent link="${parent}" />
-        <child link="${prefix}_axle_link" />
-        <xacro:insert_block name="origin" />
-        <axis xyz="0 0 1"/>
-        <dynamics friction="0.1"/>
-    </joint>
-  </xacro:macro>
+    <!-- Chassis Properties -->
+    <xacro:property name="axle_length" value="0.075" />
+    <xacro:property name="axle_height" value=".1" />
+    <xacro:property name="axle_width" value="0.075" />
+    <xacro:property name="axle_weight" value="2.45" />
+    <!-- Wheel Properties -->
+    <!-- NOTE: The below values are **guesses**-->
+    <xacro:property name="wheel_pos_x" value="-0.022"/>
+    <xacro:property name="wheel_pos_y" value="0.065"/>
+    <xacro:macro name="swerve_axle" params="prefix parent *origin">
+        <link name="${prefix}_axle_link">
+            <!-- TODO: Add intertia -->
+            <visual>
+                <origin xyz="0 0 0" rpy="0 0 0" />
+                <geometry>
+                    <mesh filename="package://swerve_description/meshes/SwerveAxle.stl" scale="0.001 0.001 0.001" />
+                </geometry>
+                <material name="blue" />
+            </visual>
+            <collision>
+                <origin xyz="0 0 0" rpy="0 0 0" />
+                <geometry>
+                    <!-- TODO: Change to a cylinder -->
+                    <box size="${axle_length} ${axle_width} ${axle_height}" />
+                </geometry>
+            </collision>
+        </link>
+        <joint name="${prefix}_axle_joint" type="continuous">
+            <parent link="${parent}" />
+            <child link="${prefix}_axle_link" />
+            <xacro:insert_block name="origin" />
+            <axis xyz="0 0 1" />
+            <dynamics friction="0.1" />
+        </joint>
+        <link name="${prefix}_wheel_link">
+            <!-- TODO: Add inertia -->
+            <visual>
+                <origin xyz="0 0 0" rpy="0 ${pi / 4} 0" />
+                <geometry>
+                    <mesh filename="package://swerve_description/meshes/SwerveWheel.stl" scale="0.001 0.001 0.001" />
+                </geometry>
+                <material name="yellow" />
+            </visual>
+            <collision>
+                <origin xyz="0 0 0" rpy="0 0 0" />
+                <geometry>
+                    <!-- TODO: Change this to a cylinder -->
+                    <box size="1 1 1" />
+                </geometry>
+            </collision>
+        </link>
+        <joint name="${prefix}_wheel_joint" type="continuous">
+            <parent link="${prefix}_axle_link" />
+            <child link="${prefix}_wheel_link" />
+            <origin xyz="${wheel_pos_x} 0 ${wheel_pos_y}" rpy="0 0 0"/>
+            <axis xyz="1 0 0" />
+            <dynamics friction="0.1" />
+        </joint>
+    </xacro:macro>
 </robot>

Commit message: added

File: src/swerve_description/urdf/parts/swerve_axle.xacro (robot description, xacro)
@@ -22,10 +22,4 @@
                 <material name="blue" />
             </visual>
-            <collision>
-                <origin xyz="0 0 0" rpy="0 0 0" />
-                <geometry>
-                    <mesh filename="package://swerve_description/meshes/SwerveAxle.stl" scale="0.001 0.001 0.001" />
-                </geometry>
-            </collision>
             <xacro:inertial_cylinder mass="${axle_mass}" radius="${axle_radius}" length="${wheel_length}" >
                 <origin xyz="0 0 0" rpy="0 0 0" />
