Commit message: Updated meshes

File: src/swerve_description/urdf/parts/square_chassis.xacro (robot description, xacro)
@@ -13,5 +13,5 @@
       </xacro:inertial_box>
       <visual>
-        <origin xyz="0 0 0" rpy="0 0 0" />
+        <origin xyz="0.061605 -0.34976 -0.53866" rpy="0 0 0" />
         <geometry>
           <mesh filename="package://swerve_description/meshes/SwerveChassis.stl" scale="0.001 0.001 0.001" />
@@ -28,5 +28,5 @@
       <parent link="base_link" />
       <child link="${prefix}_chassis_link" />
-      <origin xyz="0 0 0" rpy="0 0 0" />
+      <origin xyz="0 0 0" rpy="${pi / 2} 0 0" />
     </joint>
   </xacro:macro>

Commit message: Update chassis collision
Made a quick approximation of the robot swerve chassis for a collision model

File: src/swerve_description/urdf/parts/square_chassis.xacro (robot description, xacro)
@@ -2,8 +2,8 @@
 <robot xmlns:xacro="http://www.ros.org/wiki/xacro">
   <!-- Chassis Properties -->
-  <xacro:property name="chassis_length" value="0.18" />
-  <xacro:property name="chassis_width" value="0.33" />
-  <xacro:property name="chassis_height" value="0.135" />
-  <xacro:property name="chassis_weight" value="2.45" />
+  <xacro:property name="chassis_length" value="0.75" />
+  <xacro:property name="chassis_width" value="0.75" />
+  <xacro:property name="chassis_height" value="0.1" />
+  <xacro:property name="chassis_weight" value="10.0" />
   <xacro:macro name="square_chassis" params="prefix">
     <link name="base_link"></link>
@@ -19,7 +19,7 @@
       </visual>
       <collision>
-        <origin xyz="0 0 0" rpy="0 0 0" />
+        <origin xyz="0 ${chassis_height / 2} 0" rpy="0 0 0" />
         <geometry>
-          <box size="${chassis_length} ${chassis_width} ${chassis_height}" />
+            <box size="${chassis_length} ${chassis_height} ${chassis_width}" />
         </geometry>
       </collision>

Commit message: Added one swivel axle (no wheel)

File: src/swerve_description/urdf/parts/square_chassis.xacro (robot description, xacro)
@@ -1,8 +1,12 @@
 <?xml version="1.0"?>
 <robot xmlns:xacro="http://www.ros.org/wiki/xacro">
+<!-- Temporary color to distinguish -->
+<material name="red">
+    <color rgba="1 0 0 1"/>
+</material>
   <!-- Chassis Properties -->
-  <xacro:property name="chassis_length" value="0.18" />
-  <xacro:property name="chassis_width" value="0.33" />
-  <xacro:property name="chassis_height" value="0.135" />
+  <xacro:property name="chassis_length" value=".75" />
+  <xacro:property name="chassis_width" value="0.75" />
+  <xacro:property name="chassis_height" value=".1" />
   <xacro:property name="chassis_weight" value="2.45" />
   <xacro:macro name="square_chassis" params="prefix">
@@ -17,9 +21,10 @@
           <mesh filename="package://swerve_description/meshes/SwerveChassis.stl" scale="0.001 0.001 0.001" />
         </geometry>
+        <material name="red"/>
       </visual>
       <collision>
-        <origin xyz="0 0 0" rpy="0 0 0" />
+        <origin xyz="0 ${chassis_height / 2} 0" rpy="0 0 0" />
         <geometry>
-          <box size="${chassis_length} ${chassis_width} ${chassis_height}" />
+            <box size="${chassis_length} ${chassis_height} ${chassis_width}" />
         </geometry>
       </collision>

File: src/swerve_description/urdf/robots/swerve.urdf.xacro (robot description, xacro)
@@ -5,4 +5,11 @@
   <xacro:include filename="$(find swerve_description)/urdf/util/materials.xacro" />
   <xacro:include filename="$(find swerve_description)/urdf/parts/square_chassis.xacro" />
+  <xacro:include filename="$(find swerve_description)/urdf/parts/swerve_axle.xacro" />
+    <!-- Axle Position Variables -->
+    <xacro:property name="axle_pos" value="${301.625 / 1000}" />
+    <xacro:property name="axle_pos_y" value="${69.056 / 1000}" />
   <xacro:square_chassis prefix="swerve" />
+  <xacro:swerve_axle prefix="swerve" parent="swerve_chassis_link">
+    <origin xyz="${axle_pos} ${axle_pos_y} ${axle_pos}" rpy="${pi / 2} 0 0" />
+  </xacro:swerve_axle>
 </robot>

Commit message: Rviz configuration launch Second joint added

File: src/swerve_description/urdf/parts/square_chassis.xacro (robot description, xacro)
@@ -1,8 +1,4 @@
 <?xml version="1.0"?>
 <robot xmlns:xacro="http://www.ros.org/wiki/xacro">
-<!-- Temporary color to distinguish -->
-<material name="red">
-    <color rgba="1 0 0 1"/>
-</material>
   <!-- Chassis Properties -->
   <xacro:property name="chassis_length" value="0.75" />

File: src/swerve_description/urdf/parts/swerve_axle.xacro (robot description, xacro)
@@ -1,8 +1,4 @@
 <?xml version="1.0"?>
 <robot xmlns:xacro="http://www.ros.org/wiki/xacro">
-<!-- Temporary color to distinguish -->
-<material name="blue">
-    <color rgba="0 0 1 1"/>
-</material>
   <!-- Chassis Properties -->
   <xacro:property name="axle_length" value="0.075" />
@@ -11,5 +7,4 @@
   <xacro:property name="axle_weight" value="2.45" />
   <xacro:macro name="swerve_axle" params="prefix parent *origin">
-    <link name="base_link"></link>
     <link name="${prefix}_axle_link">
       <xacro:inertial_box mass="${axle_weight}" x="${axle_length}" y="${axle_width}" z="${axle_height}">

File: src/swerve_description/urdf/robots/swerve.urdf.xacro (robot description, xacro)
@@ -10,6 +10,15 @@
     <xacro:property name="axle_pos_y" value="${69.056 / 1000}" />
   <xacro:square_chassis prefix="swerve" />
-  <xacro:swerve_axle prefix="swerve" parent="swerve_chassis_link">
+  <xacro:swerve_axle prefix="front_left" parent="swerve_chassis_link">
     <origin xyz="${axle_pos} ${axle_pos_y} ${axle_pos}" rpy="${pi / 2} 0 0" />
   </xacro:swerve_axle>
+  <xacro:swerve_axle prefix="front_right" parent="swerve_chassis_link">
+    <origin xyz="-${axle_pos} ${axle_pos_y} ${axle_pos}" rpy="${pi / 2} 0 0" />
+  </xacro:swerve_axle>
+  <xacro:swerve_axle prefix="back_left" parent="swerve_chassis_link">
+    <origin xyz="${axle_pos} ${axle_pos_y} -${axle_pos}" rpy="${pi / 2} 0 0" />
+  </xacro:swerve_axle>
+  <xacro:swerve_axle prefix="back_right" parent="swerve_chassis_link">
+    <origin xyz="-${axle_pos} ${axle_pos_y} -${axle_pos}" rpy="${pi / 2} 0 0" />
+  </xacro:swerve_axle>
 </robot>

Commit message: fixed height error

File: src/swerve_description/urdf/parts/square_chassis.xacro (robot description, xacro)
@@ -4,5 +4,5 @@
   <xacro:property name="chassis_length" value=".7366" />
   <xacro:property name="chassis_width" value=".7366" />
-  <xacro:property name="chassis_height" value=".9" />
+  <xacro:property name="chassis_height" value="0.05588" />
   <xacro:property name="chassis_weight" value="19.0508795" />
   <xacro:macro name="square_chassis" params="prefix">

Commit message: Issue #2 #3 #5  (#13)
* Isaac extension

* Add fixes for file paths and urdf load into sim

* Add pycache to gitignore

* fixed height error

* Added collision and intertial elements to xacro

* added

* Added swerve_hardware and swerve_control

* Small change to rviz

* Changes in Extension and Xacro

* Fixed collision

Co-authored-by: Gage Miller <gagemiller155@gmail.com>

File: src/swerve_description/urdf/parts/square_chassis.xacro (robot description, xacro)
@@ -2,8 +2,8 @@
 <robot xmlns:xacro="http://www.ros.org/wiki/xacro">
   <!-- Chassis Properties -->
-  <xacro:property name="chassis_length" value="0.75" />
-  <xacro:property name="chassis_width" value="0.75" />
-  <xacro:property name="chassis_height" value="0.1" />
-  <xacro:property name="chassis_weight" value="10.0" />
+  <xacro:property name="chassis_length" value=".7366" />
+  <xacro:property name="chassis_width" value=".7366" />
+  <xacro:property name="chassis_height" value="0.05588" />
+  <xacro:property name="chassis_weight" value="19.0508795" />
   <xacro:macro name="square_chassis" params="prefix">
     <link name="base_link"></link>
@@ -20,7 +20,7 @@
       </visual>
       <collision>
-        <origin xyz="0 ${chassis_height / 2} 0" rpy="0 0 0" />
+        <origin xyz="0 ${chassis_height/2} 0" rpy="0 0 0" />
         <geometry>
-            <box size="${chassis_length} ${chassis_height} ${chassis_width}" />
+          <box size="${chassis_length} ${chassis_height} ${chassis_width}" />
         </geometry>
       </collision>

File: src/swerve_description/urdf/parts/swerve_axle.xacro (robot description, xacro)
@@ -2,15 +2,17 @@
 <robot xmlns:xacro="http://www.ros.org/wiki/xacro">
     <!-- Chassis Properties -->
-    <xacro:property name="axle_length" value="0.075" />
-    <xacro:property name="axle_height" value=".1" />
-    <xacro:property name="axle_width" value="0.075" />
-    <xacro:property name="axle_weight" value="2.45" />
+    <xacro:property name="axle_radius" value="0.075" />
+    <xacro:property name="axle_length" value=".1" />
+    <xacro:property name="axle_mass" value="0.23739" />
+    <xacro:property name="wheel_radius" value="0.0508" />
+    <xacro:property name="wheel_length" value="0.0381" />
+    <xacro:property name="wheel_mass" value="0.23133211" />
     <!-- Wheel Properties -->
     <!-- NOTE: The below values are **guesses**-->
+    <!-- NOTE: Pretty good **guesses**-->
     <xacro:property name="wheel_pos_x" value="-0.022"/>
     <xacro:property name="wheel_pos_y" value="0.065"/>
     <xacro:macro name="swerve_axle" params="prefix parent *origin">
         <link name="${prefix}_axle_link">
-            <!-- TODO: Add intertia -->
             <visual>
                 <origin xyz="0 0 0" rpy="0 0 0" />
@@ -20,11 +22,7 @@
                 <material name="blue" />
             </visual>
-            <collision>
+            <xacro:inertial_cylinder mass="${axle_mass}" radius="${axle_radius}" length="${wheel_length}" >
                 <origin xyz="0 0 0" rpy="0 0 0" />
-                <geometry>
-                    <!-- TODO: Change to a cylinder -->
-                    <box size="${axle_length} ${axle_width} ${axle_height}" />
-                </geometry>
-            </collision>
+            </xacro:inertial_cylinder>
         </link>
         <joint name="${prefix}_axle_joint" type="continuous">
@@ -36,5 +34,4 @@
         </joint>
         <link name="${prefix}_wheel_link">
-            <!-- TODO: Add inertia -->
             <visual>
                 <origin xyz="0 0 0" rpy="0 ${pi / 4} 0" />
@@ -45,10 +42,12 @@
             </visual>
             <collision>
-                <origin xyz="0 0 0" rpy="0 0 0" />
+                <origin xyz="0.021 0 0" rpy="0 ${pi / 2} 0"/>
                 <geometry>
-                    <!-- TODO: Change this to a cylinder -->
-                    <box size="1 1 1" />
+                    <cylinder  length="${wheel_length}" radius="${wheel_radius}"/>
                 </geometry>
             </collision>
+            <xacro:inertial_cylinder mass="${wheel_mass}" radius="${wheel_radius}" length="${wheel_length}" >
+                <origin xyz="0 0 0" rpy="0 ${pi / 2} 0" />
+            </xacro:inertial_cylinder>
         </link>
         <joint name="${prefix}_wheel_joint" type="continuous">
