Commit message: Elevator bot cleaning

File: src/elevator_bot_description/urdf/parts/carriage_stage.xacro (robot description, xacro)
@@ -3,6 +3,31 @@
     <!-- Carriage Properties -->
     <xacro:property name="example_property" value="-1" />
-    <xacro:macro name="carriage_stage" params="prefix">
-        <link name="carriage_stage"></link>
+    <xacro:macro name="carriage_stage" params="prefix parent origin"/>
+        <xacro:property name="length" value="0.3548888"/>
+        <xacro:property name="width" value="0.2159"/>
+        <xacro:property name="height" value="0.06985"/>
+        <xacro:property name="weight" value="0.91740145454"/>
+        <link name="${prefix}_stage_link">
+            <xacro:inertial_box mass="${weight}" x="${length}" y="${width}" z="${height}">
+                <origin xyz="0 0 0" rpy="0 0 0"/>
+            <xacro:inertial_box/>
+            <visual>
+                <origin xyz="${origin}" rpy="0 0 0"/>
+                <geometry>
+                    <mesh filename="package://elevator_bot_description/meshes/CarriageStage.stl" scale="0.001 0.001 0.001"/>
+                </geometry>
+                <material name="blue"/>
+            </visual>
+            <collision>
+                <origin xyz="0 ${height/2} 0" rpy="0 0 0"/>
+                <geometry>
+                    <box size="${length} ${width} ${height}"/>
+                </geometry>
+            </collision>
+        </link>
+        <joint name="${prefix}_stage_joint" type="fixed">
+            <parent link="${parent}"/>
+            <origin xyz="0 0 0" rpy="0 0 0"/>
+        </joint>
     </xacro:macro>
 </robot>

Commit message: Still broken, but now xacro works, which is pog

File: src/elevator_bot_description/urdf/parts/carriage_stage.xacro (robot description, xacro)
@@ -2,6 +2,6 @@
 <robot xmlns:xacro="http://www.ros.org/wiki/xacro">
     <!-- Carriage Properties -->
-    <xacro:property name="example_property" value="-1" />
-    <xacro:macro name="carriage_stage" params="prefix parent origin"/>
+    <!-- <xacro:property name="example_property" value="-1" /> -->
+    <xacro:macro name="carriage_stage" params="prefix parent origin">
         <xacro:property name="length" value="0.3548888"/>
         <xacro:property name="width" value="0.2159"/>
@@ -11,5 +11,5 @@
             <xacro:inertial_box mass="${weight}" x="${length}" y="${width}" z="${height}">
                 <origin xyz="0 0 0" rpy="0 0 0"/>
-            <xacro:inertial_box/>
+            </xacro:inertial_box>
             <visual>
                 <origin xyz="${origin}" rpy="0 0 0"/>

File: src/elevator_bot_description/urdf/parts/second_stage.xacro (robot description, xacro)
@@ -6,29 +6,30 @@
     <!-- 47in (1.1938m) length total -->
     <!-- 4.9748lbs (2.2565kgs) weight total -->
+    <xacro:property name="total_length" value="1.1938" />
+    <xacro:property name="total_width" value="0.3937" />
+    <xacro:property name="total_height" value="0.0508" /> <!-- Not completely accurate!-->
+    <xacro:property name="total_weight" value="2.2565" />
+    <xacro:property name="bar_height" value="0.0508" />
+    <xacro:property name="bar_width" value="0.0254" />
     <xacro:macro name="second_stage" params="prefix">
         <!-- Second Stage Properties -->
-        <link name="second_stage"></link>
-        <xacro:property name="total_length" value="1.1938" />
-        <xacro:property name="total_width" value="0.3937" />
-        <xacro:property name="total_height" value="0.0508" /> <!-- Not completely accurate!-->
-        <xacro:property name="weight" value="2.2565" />
-        <xacro:property name="bar_height" value="0.0508" />
-        <xacro:property name="bar_width" value="0.0254" />
-        <xacro:inertial_box mass="${total_weight}" x="${total_length}" y="${total_width}" z="${total_height}">
-            <origin xyz="0 0 0" rpy="0 0 0" />
-        </xacro:inertial_box>
-        <visual>
-            <origin xyz="0 0 0" rpy="0 0 0" />
-            <geometry>
-                <mesh filename="package://elevator_bot_description/meshes/2ndStageStructure.stl" scale="0.1 0.1 0.1"/>
-            </geometry>
-            <material name="blue" />
-        </visual>
-        <collision>
-            <origin xyz="0 ${total_height/2} 0" rpy="0 0 0" />
-            <geometry>
-                <box size="${total_length} ${total_height} ${total_width}" />
-            </geometry>
-        </collision>
+        <link name="second_stage">
+            <xacro:inertial_box mass="${total_weight}" x="${total_length}" y="${total_width}" z="${total_height}">
+                <origin xyz="0 0 0" rpy="0 0 0" />
+            </xacro:inertial_box>
+            <visual>
+                <origin xyz="0.061605 -0.75 -0.53866" rpy="0 0 0" />
+                <geometry>
+                    <mesh filename="package://elevator_bot_description/meshes/2ndStageStructure.stl" scale="0.001 0.001 0.001" />
+                </geometry>
+                <material name="blue" />
+            </visual>
+            <collision>
+                <origin xyz="0 ${total_height/2} 0" rpy="0 0 0" />
+                <geometry>
+                    <box size="${total_length} ${total_height} ${total_width}" />
+                </geometry>
+            </collision>
+        </link>
     </xacro:macro>
 </robot>

File: src/elevator_bot_description/urdf/robots/elevator_bot.urdf.xacro (robot description, xacro)
@@ -2,10 +2,14 @@
 <robot name="elevator_bot" xmlns:xacro="http://www.ros.org/wiki/xacro">
     <!-- Include Files -->
-    <xacro:include filename="$(find elevator_bot_description)/urdf/parts/base_stage.xacro" />
-    <xacro:include filename="$(find elevator_bot_description)/urdf/parts/carriage_stage.xacro" />
+    <!-- <xacro:include filename="$(find elevator_bot_description)/urdf/parts/base_stage.xacro" /> -->
+    <!-- <xacro:include filename="$(find elevator_bot_description)/urdf/parts/carriage_stage.xacro" /> -->
     <xacro:include filename="$(find elevator_bot_description)/urdf/parts/second_stage.xacro" />
+    <xacro:include filename="$(find elevator_bot_description)/urdf/util/macros.xacro" />
+    <xacro:include filename="$(find elevator_bot_description)/urdf/util/materials.xacro" />
     <!-- Position Variables -->
-    <xacro:base_stage prefix="elevator_bot" />
-    <xacro:second_stage parent="elevator_bot_base_stage" />
-    <xacro:carriage_stage parent="elevator_bot_second_stage" />
+    <!-- <xacro:base_stage prefix="elevator_bot" /> -->
+    <xacro:second_stage prefix="elevator_bot"/>
+    <!-- <xacro:carriage_stage parent="elevator_bot_second_stage">
+        <origin xyz="0 0 0"></origin>
+    </xacro:carriage_stage> -->
 </robot>
