Commit message: completely broken stuff :)

File: src/elevator_bot_description/urdf/parts/second_stage.xacro (robot description, xacro)
@@ -1,8 +1,34 @@
 <?xml version="1.0"?>
 <robot xmlns:xacro="http://www.ros.org/wiki/xacro">
-    <!-- Second Stage Properties -->
-    <xacro:property name="example_property" value="-1" />
+    <!-- 2in (0.0508m) line height -->
+    <!-- 1in (0.0254m) line width -->
+    <!-- 15.5 (0.3937m) width total -->
+    <!-- 47in (1.1938m) length total -->
+    <!-- 4.9748lbs (2.2565kgs) weight total -->
     <xacro:macro name="second_stage" params="prefix">
+        <!-- Second Stage Properties -->
         <link name="second_stage"></link>
+        <xacro:property name="total_length" value="1.1938" />
+        <xacro:property name="total_width" value="0.3937" />
+        <xacro:property name="total_height" value="0.0508" /> <!-- Not completely accurate!-->
+        <xacro:property name="weight" value="2.2565" />
+        <xacro:property name="bar_height" value="0.0508" />
+        <xacro:property name="bar_width" value="0.0254" />
+        <xacro:inertial_box mass="${total_weight}" x="${total_length}" y="${total_width}" z="${total_height}">
+            <origin xyz="0 0 0" rpy="0 0 0" />
+        </xacro:inertial_box>
+        <visual>
+            <origin xyz="0 0 0" rpy="0 0 0" />
+            <geometry>
+                <mesh filename="package://elevator_bot_description/meshes/2ndStageStructure.stl" scale="0.1 0.1 0.1"/>
+            </geometry>
+            <material name="blue" />
+        </visual>
+        <collision>
+            <origin xyz="0 ${total_height/2} 0" rpy="0 0 0" />
+            <geometry>
+                <box size="${total_length} ${total_height} ${total_width}" />
+            </geometry>
+        </collision>
     </xacro:macro>
 </robot>

File: src/elevator_bot_description/urdf/robots/elevator_bot.urdf.xacro (robot description, xacro)
@@ -1,5 +1,11 @@
 <?xml version="1.0"?>
-<robot name="swerve" xmlns:xacro="http://www.ros.org/wiki/xacro">
+<robot name="elevator_bot" xmlns:xacro="http://www.ros.org/wiki/xacro">
     <!-- Include Files -->
+    <xacro:include filename="$(find elevator_bot_description)/urdf/parts/base_stage.xacro" />
+    <xacro:include filename="$(find elevator_bot_description)/urdf/parts/carriage_stage.xacro" />
+    <xacro:include filename="$(find elevator_bot_description)/urdf/parts/second_stage.xacro" />
     <!-- Position Variables -->
+    <xacro:base_stage prefix="elevator_bot" />
+    <xacro:second_stage parent="elevator_bot_base_stage" />
+    <xacro:carriage_stage parent="elevator_bot_second_stage" />
 </robot>

Commit message: Patched Models + Second_Stage - Patched models (@Nithin) - Created collision for second_stage

File: src/elevator_bot_description/urdf/parts/second_stage.xacro (robot description, xacro)
@@ -6,29 +6,43 @@
     <!-- 47in (1.1938m) length total -->
     <!-- 4.9748lbs (2.2565kgs) weight total -->
-    <!-- DEBUG: Define a material that's transparent to help line up the collision box -->
-    <material name="grey_overlay">
-        <color rgba="0.2 0.2 0.2 0.5" />
-      </material>
-    <xacro:property name="total_length" value="1.1938" />
-    <xacro:property name="total_width" value="0.3937" />
-    <xacro:property name="total_height" value="0.0508" /> <!-- Not completely accurate!-->
+    <!-- These are more measurement guesses because the measured size is being weird -->
+    <xacro:property name="total_height" value="1.525" />
+    <xacro:property name="total_width" value="0.485" /> <!-- 0.53333 -->
+    <xacro:property name="total_length" value="0.0508" />
     <xacro:property name="total_weight" value="2.2565" />
-    <xacro:property name="bar_height" value="0.0508" />
+    <xacro:property name="bar_height" value="0.0265" />
     <xacro:property name="bar_width" value="0.0254" />
     <xacro:macro name="second_stage" params="prefix">
-        <!-- Second Stage Properties -->
         <link name="second_stage">
-            <xacro:inertial_box mass="${total_weight}" x="${total_length}" y="${total_width}" z="${total_height}">
+            <xacro:inertial_box mass="${total_weight}" x="${total_height}" y="${total_width}" z="${total_length}">
                 <origin xyz="0 0 0" rpy="0 0 0" />
             </xacro:inertial_box>
-            <collision> <!-- Does not work! -->
-                <origin xyz="0 0 ${2*total_height}" rpy="0 0 0" />
+            <!-- All values here are completely made up. For your own sake, don't try to understand them -->
+            <collision> <!-- Top Bar -->
+                <origin xyz="0 0 ${total_height-bar_height/2+0.001}" rpy="0 0 0" />
                 <geometry>
-                    <box size="${total_length} ${total_width} ${total_height}" />
+                    <box size="${total_width} ${total_length} ${bar_height}"/>
                 </geometry>
-                <material name="blue" />
+            </collision>
+            <collision> <!-- Bottom Bar -->
+                <origin xyz="0 0 ${bar_height/2+0.001}" rpy="0 0 0" />
+                <geometry>
+                    <box size="${total_width} ${total_length} ${bar_height}"/>
+                </geometry>
+            </collision>
+            <collision> <!-- Left Bar -->
+                <origin xyz="${-total_width/2-bar_width/2+0.001} 0 ${total_height/2+0.001}" rpy="0 0 0" />
+                <geometry>
+                    <box size="${bar_width} ${total_length} ${total_height}"/>
+                </geometry>
+            </collision>
+            <collision> <!-- Right Bar -->
+                <origin xyz="${total_width/2+bar_width/2-0.001} 0 ${total_height/2+0.001}" rpy="0 0 0" />
+                <geometry>
+                    <box size="${bar_width} ${total_length} ${total_height}"/>
+                </geometry>
             </collision>
             <visual>
-                <origin xyz=".5 ${-4/3} ${-2/3}" rpy="0 0 0" /> <!-- Origin is offset to center the model, if there are problems, reset this to 0 0 0 -->
+                <origin xyz="${-50/123} ${-total_length/2} ${-1/16}" rpy="0 0 0" /> <!-- The model is *very slightly offset, even with @Nithin's model changes -->
                 <geometry>
                     <mesh filename="package://elevator_bot_description/meshes/2ndStageStructure.stl" scale="0.001 0.001 0.001" />
@@ -37,14 +51,4 @@
             </visual>
         </link>
-        <!-- DEBUG: A separate part to help line up the collision with the model -->
-        <link name="temporary_box">
-            <visual>
-                <origin xyz="0 0 ${11*total_height}" rpy="0 0 0" />
-                <geometry>
-                    <box size="${total_width} ${total_height} ${total_length}" />
-                </geometry>
-                <material name="grey_overlay" />
-            </visual>
-        </link>
     </xacro:macro>
 </robot>

File: src/elevator_bot_description/urdf/robots/elevator_bot.urdf.xacro (robot description, xacro)
@@ -8,5 +8,5 @@
     <xacro:include filename="$(find elevator_bot_description)/urdf/util/materials.xacro" />
     <!-- Parts of the robot -->
-    <xacro:base_stage prefix="elevator_bot" />
+    <!-- <xacro:base_stage prefix="elevator_bot" /> -->
     <xacro:second_stage prefix="elevator_bot"/>
     <!-- <xacro:carriage_stage /> -->
