Commit message: Some debug changes - Added debug overlay to second_stage - Filled out a more complete template for base_stage - Hacky solution to fix the offset (should be reverted once the models get pushed)

File: src/elevator_bot_description/urdf/parts/base_stage.xacro (robot description, xacro)
@@ -1,8 +1,32 @@
 <?xml version="1.0"?>
 <robot xmlns:xacro="http://www.ros.org/wiki/xacro">
-    <!-- Base Stage Properties -->
-    <xacro:property name="example_property" value="-1" />
+    <!-- PLACEHOLDER VALUES! CHANGE THESE -->
+    <xacro:property name="total_length" value="1" />
+    <xacro:property name="total_width" value="1" />
+    <xacro:property name="total_height" value="1" />
+    <xacro:property name="total_weight" value="1" />
+    <xacro:property name="bar_height" value="1" />
+    <xacro:property name="bar_width" value="1" />
+    <!-- This entire file is pretty much a placeholder -->
+    <!-- Feel free to delete everything and start over -->
     <xacro:macro name="base_stage" params="prefix">
-        <link name="base_stage"></link>
+        <link name="base_stage">
+            <xacro:inertial_box mass="${total_weight}" x="${total_length}" y="${total_width}" z="${total_height}">
+                <origin xyz="0 0 0" rpy="0 0 0" />
+            </xacro:inertial_box>
+            <visual>
+                <origin xyz="-1 -.5 0" rpy="0 0 0" />
+                <geometry>
+                    <mesh filename="package://elevator_bot_description/meshes/BaseStageStructure.stl" scale="0.001 0.001 0.001" />
+                </geometry>
+                <material name="blue" />
+            </visual>
+            <collision>
+                <origin xyz="0 ${total_height/2} 0" rpy="0 0 0" />
+                <geometry>
+                    <box size="${total_length} ${total_height} ${total_width}" />
+                </geometry>
+            </collision>
+        </link>
     </xacro:macro>
 </robot>

File: src/elevator_bot_description/urdf/parts/second_stage.xacro (robot description, xacro)
@@ -6,4 +6,8 @@
     <!-- 47in (1.1938m) length total -->
     <!-- 4.9748lbs (2.2565kgs) weight total -->
+    <!-- DEBUG: Define a material that's transparent to help line up the collision box -->
+    <material name="grey_overlay">
+        <color rgba="0.2 0.2 0.2 0.5" />
+      </material>
     <xacro:property name="total_length" value="1.1938" />
     <xacro:property name="total_width" value="0.3937" />
@@ -18,6 +22,13 @@
                 <origin xyz="0 0 0" rpy="0 0 0" />
             </xacro:inertial_box>
+            <collision> <!-- Does not work! -->
+                <origin xyz="0 0 ${2*total_height}" rpy="0 0 0" />
+                <geometry>
+                    <box size="${total_length} ${total_width} ${total_height}" />
+                </geometry>
+                <material name="blue" />
+            </collision>
             <visual>
-                <origin xyz="0.061605 -0.75 -0.53866" rpy="0 0 0" />
+                <origin xyz=".5 ${-4/3} ${-2/3}" rpy="0 0 0" /> <!-- Origin is offset to center the model, if there are problems, reset this to 0 0 0 -->
                 <geometry>
                     <mesh filename="package://elevator_bot_description/meshes/2ndStageStructure.stl" scale="0.001 0.001 0.001" />
@@ -25,10 +36,14 @@
                 <material name="blue" />
             </visual>
-            <collision>
-                <origin xyz="0 ${total_height/2} 0" rpy="0 0 0" />
+        </link>
+        <!-- DEBUG: A separate part to help line up the collision with the model -->
+        <link name="temporary_box">
+            <visual>
+                <origin xyz="0 0 ${11*total_height}" rpy="0 0 0" />
                 <geometry>
-                    <box size="${total_length} ${total_height} ${total_width}" />
+                    <box size="${total_width} ${total_height} ${total_length}" />
                 </geometry>
-            </collision>
+                <material name="grey_overlay" />
+            </visual>
         </link>
     </xacro:macro>

File: src/elevator_bot_description/urdf/robots/elevator_bot.urdf.xacro (robot description, xacro)
@@ -2,14 +2,12 @@
 <robot name="elevator_bot" xmlns:xacro="http://www.ros.org/wiki/xacro">
     <!-- Include Files -->
-    <!-- <xacro:include filename="$(find elevator_bot_description)/urdf/parts/base_stage.xacro" /> -->
-    <!-- <xacro:include filename="$(find elevator_bot_description)/urdf/parts/carriage_stage.xacro" /> -->
+    <xacro:include filename="$(find elevator_bot_description)/urdf/parts/base_stage.xacro" />
+    <xacro:include filename="$(find elevator_bot_description)/urdf/parts/carriage_stage.xacro" />
     <xacro:include filename="$(find elevator_bot_description)/urdf/parts/second_stage.xacro" />
     <xacro:include filename="$(find elevator_bot_description)/urdf/util/macros.xacro" />
     <xacro:include filename="$(find elevator_bot_description)/urdf/util/materials.xacro" />
-    <!-- Position Variables -->
-    <!-- <xacro:base_stage prefix="elevator_bot" /> -->
+    <!-- Parts of the robot -->
+    <xacro:base_stage prefix="elevator_bot" />
     <xacro:second_stage prefix="elevator_bot"/>
-    <!-- <xacro:carriage_stage parent="elevator_bot_second_stage">
-        <origin xyz="0 0 0"></origin>
-    </xacro:carriage_stage> -->
+    <!-- <xacro:carriage_stage /> -->
 </robot>

Commit message: Centered mesh, updated joints, second stage error

File: src/elevator_bot_description/urdf/parts/base_stage.xacro (robot description, xacro)
@@ -11,10 +11,11 @@
     <!-- Feel free to delete everything and start over -->
     <xacro:macro name="base_stage" params="prefix">
-        <link name="base_stage">
+        <link name="base_link"></link>
+        <link name="base_stage_link">
             <xacro:inertial_box mass="${total_weight}" x="${total_length}" y="${total_width}" z="${total_height}">
                 <origin xyz="0 0 0" rpy="0 0 0" />
             </xacro:inertial_box>
             <visual>
-                <origin xyz="-1 -.5 0" rpy="0 0 0" />
+                <origin  xyz="0 0 ${total_height/2}" rpy="0 -${pi/2} -${pi/2}"  />
                 <geometry>
                     <mesh filename="package://elevator_bot_description/meshes/BaseStageStructure.stl" scale="0.001 0.001 0.001" />
@@ -23,5 +24,5 @@
             </visual>
             <collision>
-                <origin xyz="0 ${total_height/2} 0" rpy="0 0 0" />
+                <origin xyz="0 0 0" rpy="0 0 0" />
                 <geometry>
                     <box size="${total_length} ${total_height} ${total_width}" />
@@ -29,4 +30,14 @@
             </collision>
         </link>
+        <joint name="base_stage_joint" type="fixed">
+            <parent link="base_link" />
+            <child link="base_stage_link" />
+            <origin xyz="0 0 0" rpy="0 0 0" />
+        </joint>
+        <joint name="base_stage_joint" type="prismatic">
+            <parent link="base_stage_link"/>
+            <child link="second_stage_link" />
+            <origin xyz="0 0 0" rpy="0 0 0"/>
+        </joint>
     </xacro:macro>
 </robot>

File: src/elevator_bot_description/urdf/parts/carriage_stage.xacro (robot description, xacro)
@@ -3,5 +3,5 @@
     <!-- Carriage Properties -->
     <!-- <xacro:property name="example_property" value="-1" /> -->
-    <xacro:macro name="carriage_stage" params="prefix parent origin">
+    <xacro:macro name="carriage_stage" params="prefix">
         <xacro:property name="length" value="0.3548888"/>
         <xacro:property name="width" value="0.2159"/>
@@ -13,5 +13,5 @@
             </xacro:inertial_box>
             <visual>
-                <origin xyz="${origin}" rpy="0 0 0"/>
+                <origin xyz="0 0 0" rpy="0 0 0"/>
                 <geometry>
                     <mesh filename="package://elevator_bot_description/meshes/CarriageStage.stl" scale="0.001 0.001 0.001"/>
@@ -26,8 +26,4 @@
             </collision>
         </link>
-        <joint name="${prefix}_stage_joint" type="fixed">
-            <parent link="${parent}"/>
-            <origin xyz="0 0 0" rpy="0 0 0"/>
-        </joint>
     </xacro:macro>
 </robot>

File: src/elevator_bot_description/urdf/parts/second_stage.xacro (robot description, xacro)
@@ -14,5 +14,5 @@
     <xacro:property name="bar_width" value="0.0254" />
     <xacro:macro name="second_stage" params="prefix">
-        <link name="second_stage">
+        <link name="second_stage_link">
             <xacro:inertial_box mass="${total_weight}" x="${total_height}" y="${total_width}" z="${total_length}">
                 <origin xyz="0 0 0" rpy="0 0 0" />
@@ -51,4 +51,9 @@
             </visual>
         </link>
+        <joint name="second_stage_joint" type="prismatic">
+            <parent link="second_stage_link"/>
+            <child link="carriage_stage_link" />
+            <origin xyz="0 0 0" rpy="0 0 0"/>
+        </joint>
     </xacro:macro>
 </robot>

File: src/elevator_bot_description/urdf/robots/elevator_bot.urdf.xacro (robot description, xacro)
@@ -8,6 +8,6 @@
     <xacro:include filename="$(find elevator_bot_description)/urdf/util/materials.xacro" />
     <!-- Parts of the robot -->
-    <xacro:base_stage prefix="elevator_bot" />
-    <xacro:second_stage prefix="elevator_bot" parent="base_stage"/>
-    <xacro:carriage_stage prefix="elevator_bot" parent="second_stage"/>
+    <xacro:base_stage prefix="base" />
+    <xacro:second_stage prefix="second" />
+    <xacro:carriage_stage prefix="carriage"/>
 </robot>
