Commit message: Added collision and intertial elements to xacro

File: src/swerve_description/swerve.urdf (robot description, URDF)
Before this commit: robot swerve, 10 links, 9 joints
Links:
- link back_left_axle_link: mass None -> 0.23739; geometry collision mesh filename=package://swerve_description/meshes/SwerveAxle.stl scale=0.001 0.001 0.001; visual mesh filename=package://swerve_description/meshes/SwerveAxle.stl scale=0.001 0.001 0.001
- link back_left_wheel_link: mass None -> 0.23133211; geometry collision cylinder length=0.0381 radius=0.0508; visual mesh filename=package://swerve_description/meshes/SwerveWheel.stl scale=0.001 0.001 0.001
- link back_right_axle_link: mass None -> 0.23739; geometry collision mesh filename=package://swerve_description/meshes/SwerveAxle.stl scale=0.001 0.001 0.001; visual mesh filename=package://swerve_description/meshes/SwerveAxle.stl scale=0.001 0.001 0.001
- link back_right_wheel_link: mass None -> 0.23133211; geometry collision cylinder length=0.0381 radius=0.0508; visual mesh filename=package://swerve_description/meshes/SwerveWheel.stl scale=0.001 0.001 0.001
- link front_left_axle_link: mass None -> 0.23739; geometry collision mesh filename=package://swerve_description/meshes/SwerveAxle.stl scale=0.001 0.001 0.001; visual mesh filename=package://swerve_description/meshes/SwerveAxle.stl scale=0.001 0.001 0.001
- link front_left_wheel_link: mass None -> 0.23133211; geometry collision cylinder length=0.0381 radius=0.0508; visual mesh filename=package://swerve_description/meshes/SwerveWheel.stl scale=0.001 0.001 0.001
- link front_right_axle_link: mass None -> 0.23739; geometry collision mesh filename=package://swerve_description/meshes/SwerveAxle.stl scale=0.001 0.001 0.001; visual mesh filename=package://swerve_description/meshes/SwerveAxle.stl scale=0.001 0.001 0.001
- link front_right_wheel_link: mass None -> 0.23133211; geometry collision cylinder length=0.0381 radius=0.0508; visual mesh filename=package://swerve_description/meshes/SwerveWheel.stl scale=0.001 0.001 0.001
- link swerve_chassis_link: mass 10.0 -> 19.0508795; geometry collision mesh filename=package://swerve_description/meshes/contact_mesh_chasis.stl scale=0.001 0.001 0.001; visual mesh filename=package://swerve_description/meshes/SwerveChassis.stl scale=0.001 0.001 0.001

File: src/swerve_description/urdf/parts/square_chassis.xacro (robot description, xacro)
@@ -2,8 +2,8 @@
 <robot xmlns:xacro="http://www.ros.org/wiki/xacro">
   <!-- Chassis Properties -->
-  <xacro:property name="chassis_length" value="0.75" />
-  <xacro:property name="chassis_width" value="0.75" />
-  <xacro:property name="chassis_height" value="0.1" />
-  <xacro:property name="chassis_weight" value="10.0" />
+  <xacro:property name="chassis_length" value=".7366" />
+  <xacro:property name="chassis_width" value=".7366" />
+  <xacro:property name="chassis_height" value=".9" />
+  <xacro:property name="chassis_weight" value="19.0508795" />
   <xacro:macro name="square_chassis" params="prefix">
     <link name="base_link"></link>
@@ -20,7 +20,7 @@
       </visual>
       <collision>
-        <origin xyz="0 ${chassis_height / 2} 0" rpy="0 0 0" />
+        <origin xyz="${-chassis_length/2} -0.005 ${-chassis_width/2}" rpy="0 0 0" />
         <geometry>
-            <box size="${chassis_length} ${chassis_height} ${chassis_width}" />
+            <mesh filename="package://swerve_description/meshes/contact_mesh_chasis.stl" scale="0.001 0.001 0.001" />
         </geometry>
       </collision>

File: src/swerve_description/urdf/parts/swerve_axle.xacro (robot description, xacro)
@@ -2,15 +2,17 @@
 <robot xmlns:xacro="http://www.ros.org/wiki/xacro">
     <!-- Chassis Properties -->
-    <xacro:property name="axle_length" value="0.075" />
-    <xacro:property name="axle_height" value=".1" />
-    <xacro:property name="axle_width" value="0.075" />
-    <xacro:property name="axle_weight" value="2.45" />
+    <xacro:property name="axle_radius" value="0.075" />
+    <xacro:property name="axle_length" value=".1" />
+    <xacro:property name="axle_mass" value="0.23739" />
+    <xacro:property name="wheel_radius" value="0.0508" />
+    <xacro:property name="wheel_length" value="0.0381" />
+    <xacro:property name="wheel_mass" value="0.23133211" />
     <!-- Wheel Properties -->
     <!-- NOTE: The below values are **guesses**-->
+    <!-- NOTE: Pretty good **guesses**-->
     <xacro:property name="wheel_pos_x" value="-0.022"/>
     <xacro:property name="wheel_pos_y" value="0.065"/>
     <xacro:macro name="swerve_axle" params="prefix parent *origin">
         <link name="${prefix}_axle_link">
-            <!-- TODO: Add intertia -->
             <visual>
                 <origin xyz="0 0 0" rpy="0 0 0" />
@@ -23,8 +25,10 @@
                 <origin xyz="0 0 0" rpy="0 0 0" />
                 <geometry>
-                    <!-- TODO: Change to a cylinder -->
-                    <box size="${axle_length} ${axle_width} ${axle_height}" />
+                    <mesh filename="package://swerve_description/meshes/SwerveAxle.stl" scale="0.001 0.001 0.001" />
                 </geometry>
             </collision>
+            <xacro:inertial_cylinder mass="${axle_mass}" radius="${axle_radius}" length="${wheel_length}" >
+                <origin xyz="0 0 0" rpy="0 0 0" />
+            </xacro:inertial_cylinder>
         </link>
         <joint name="${prefix}_axle_joint" type="continuous">
@@ -36,5 +40,4 @@
         </joint>
         <link name="${prefix}_wheel_link">
-            <!-- TODO: Add inertia -->
             <visual>
                 <origin xyz="0 0 0" rpy="0 ${pi / 4} 0" />
@@ -45,10 +48,12 @@
             </visual>
             <collision>
-                <origin xyz="0 0 0" rpy="0 0 0" />
+                <origin xyz="0.021 0 0" rpy="0 ${pi / 2} 0"/>
                 <geometry>
-                    <!-- TODO: Change this to a cylinder -->
-                    <box size="1 1 1" />
+                    <cylinder  length="${wheel_length}" radius="${wheel_radius}"/>
                 </geometry>
             </collision>
+            <xacro:inertial_cylinder mass="${wheel_mass}" radius="${wheel_radius}" length="${wheel_length}" >
+                <origin xyz="0 0 0" rpy="0 ${pi / 2} 0" />
+            </xacro:inertial_cylinder>
         </link>
         <joint name="${prefix}_wheel_joint" type="continuous">

Commit message: Added swerve_hardware and swerve_control

File: src/swerve_description/swerve.urdf (robot description, URDF)
Before this commit: robot swerve, 10 links, 9 joints
Links:
- link back_left_axle_link: geometry visual mesh filename=package://swerve_description/meshes/SwerveAxle.stl scale=0.001 0.001 0.001
- link back_right_axle_link: geometry visual mesh filename=package://swerve_description/meshes/SwerveAxle.stl scale=0.001 0.001 0.001
- link front_left_axle_link: geometry visual mesh filename=package://swerve_description/meshes/SwerveAxle.stl scale=0.001 0.001 0.001
- link front_right_axle_link: geometry visual mesh filename=package://swerve_description/meshes/SwerveAxle.stl scale=0.001 0.001 0.001

Commit message: Fixed collision

File: src/swerve_description/swerve.urdf (robot description, URDF)
Before this commit: robot swerve, 10 links, 9 joints
Links:
- link swerve_chassis_link: geometry collision box size=0.7366 0.05588 0.7366; visual mesh filename=package://swerve_description/meshes/SwerveChassis.stl scale=0.001 0.001 0.001

File: src/swerve_description/urdf/parts/square_chassis.xacro (robot description, xacro)
@@ -20,7 +20,7 @@
       </visual>
       <collision>
-        <origin xyz="${-chassis_length/2} -0.005 ${-chassis_width/2}" rpy="0 0 0" />
+        <origin xyz="0 ${chassis_height/2} 0" rpy="0 0 0" />
         <geometry>
-            <mesh filename="package://swerve_description/meshes/contact_mesh_chasis.stl" scale="0.001 0.001 0.001" />
+          <box size="${chassis_length} ${chassis_height} ${chassis_width}" />
         </geometry>
       </collision>

Commit message: added collision to axle

File: src/swerve_description/swerve.urdf (robot description, URDF)
Before this commit: robot swerve, 10 links, 9 joints
Links:
- link back_left_axle_link: geometry collision cylinder length=0.05 radius=0.05; visual mesh filename=package://swerve_description/meshes/SwerveAxle.stl scale=0.001 0.001 0.001
- link back_right_axle_link: geometry collision cylinder length=0.05 radius=0.05; visual mesh filename=package://swerve_description/meshes/SwerveAxle.stl scale=0.001 0.001 0.001
- link front_left_axle_link: geometry collision cylinder length=0.05 radius=0.05; visual mesh filename=package://swerve_description/meshes/SwerveAxle.stl scale=0.001 0.001 0.001
- link front_right_axle_link: geometry collision cylinder length=0.05 radius=0.05; visual mesh filename=package://swerve_description/meshes/SwerveAxle.stl scale=0.001 0.001 0.001

File: src/swerve_description/urdf/parts/swerve_axle.xacro (robot description, xacro)
@@ -22,4 +22,10 @@
                 <material name="blue" />
             </visual>
+            <collision>
+                <origin xyz="0 0 0" rpy="0 0 0"/>
+                <geometry>
+                    <cylinder  length="${axle_length/2}" radius="0.05"/>
+                </geometry>
+            </collision>
             <xacro:inertial_cylinder mass="${axle_mass}" radius="${axle_radius}" length="${wheel_length}" >
                 <origin xyz="0 0 0" rpy="0 0 0" />

Commit message: Fixed naming rear and back; made constant turning

File: src/swerve_description/swerve.urdf (robot description, URDF)
Before this commit: robot swerve, 10 links, 9 joints
Links:
- removed link back_left_axle_link
- removed link back_left_wheel_link
- removed link back_right_axle_link
- removed link back_right_wheel_link
- added link rear_left_axle_link, mass 0.23739; visual mesh filename=package://swerve_description/meshes/SwerveAxle.stl scale=0.001 0.001 0.001
- added link rear_left_wheel_link, mass 0.23133211; collision cylinder length=0.0381 radius=0.0508; visual mesh filename=package://swerve_description/meshes/SwerveWheel.stl scale=0.001 0.001 0.001
- added link rear_right_axle_link, mass 0.23739; visual mesh filename=package://swerve_description/meshes/SwerveAxle.stl scale=0.001 0.001 0.001
- added link rear_right_wheel_link, mass 0.23133211; collision cylinder length=0.0381 radius=0.0508; visual mesh filename=package://swerve_description/meshes/SwerveWheel.stl scale=0.001 0.001 0.001
Joints:
- removed joint back_left_axle_joint
- removed joint back_left_wheel_joint
- removed joint back_right_axle_joint
- removed joint back_right_wheel_joint
- added joint rear_left_axle_joint: type continuous, parent swerve_chassis_link, child rear_left_axle_link, origin xyz=0.301625 0.06905599999999999 -0.301625 rpy=1.5707963267948966 0 0, axis 0 0 1
- added joint rear_left_wheel_joint: type continuous, parent rear_left_axle_link, child rear_left_wheel_link, origin xyz=-0.022 0 0.065 rpy=0 0 0, axis 1 0 0
- added joint rear_right_axle_joint: type continuous, parent swerve_chassis_link, child rear_right_axle_link, origin xyz=-0.301625 0.06905599999999999 -0.301625 rpy=1.5707963267948966 0 0, axis 0 0 1
- added joint rear_right_wheel_joint: type continuous, parent rear_right_axle_link, child rear_right_wheel_link, origin xyz=-0.022 0 0.065 rpy=0 0 0, axis 1 0 0

File: src/swerve_description/urdf/control/drive.xacro (robot description, xacro)
@@ -16,5 +16,5 @@
         <state_interface name="velocity"/>
       </joint>
-      <joint name="back_left_wheel_joint">
+      <joint name="rear_left_wheel_joint">
         <command_interface name="velocity">
           <param name="min">-1</param>
@@ -32,5 +32,5 @@
         <state_interface name="velocity"/>
       </joint>
-      <joint name="back_right_wheel_joint">
+      <joint name="rear_right_wheel_joint">
         <command_interface name="velocity">
           <param name="min">-1</param>
@@ -48,5 +48,5 @@
         <state_interface name="velocity"/>
       </joint>
-      <joint name="back_left_axle_joint">
+      <joint name="rear_left_axle_joint">
         <command_interface name="velocity">
           <param name="min">-1</param>
@@ -64,5 +64,5 @@
         <state_interface name="velocity"/>
       </joint>
-      <joint name="back_right_axle_joint">
+      <joint name="rear_right_axle_joint">
         <command_interface name="velocity">
           <param name="min">-1</param>

File: src/swerve_description/urdf/robots/swerve.urdf.xacro (robot description, xacro)
@@ -19,8 +19,8 @@
     <origin xyz="-${axle_pos} ${axle_pos_y} ${axle_pos}" rpy="${pi / 2} 0 0" />
   </xacro:swerve_axle>
-  <xacro:swerve_axle prefix="back_left" parent="swerve_chassis_link">
+  <xacro:swerve_axle prefix="rear_left" parent="swerve_chassis_link">
     <origin xyz="${axle_pos} ${axle_pos_y} -${axle_pos}" rpy="${pi / 2} 0 0" />
   </xacro:swerve_axle>
-  <xacro:swerve_axle prefix="back_right" parent="swerve_chassis_link">
+  <xacro:swerve_axle prefix="rear_right" parent="swerve_chassis_link">
     <origin xyz="-${axle_pos} ${axle_pos_y} -${axle_pos}" rpy="${pi / 2} 0 0" />
   </xacro:swerve_axle>

Commit message: LOADS INTO ISAAC SIM WITHOUT ERRORS (flying robot)

File: src/swerve_description/swerve.urdf (robot description, URDF)
Before this commit: robot swerve, 10 links, 9 joints
Links:
- removed link back_left_axle_link
- removed link back_left_wheel_link
- removed link back_right_axle_link
- removed link back_right_wheel_link
- added link rear_left_axle_link, mass 0.23739; collision cylinder length=0.05 radius=0.05; visual mesh filename=package://swerve_description/meshes/SwerveAxle.stl scale=0.001 0.001 0.001
- added link rear_left_wheel_link, mass 0.23133211; collision cylinder length=0.0381 radius=0.0508; visual mesh filename=package://swerve_description/meshes/SwerveWheel.stl scale=0.001 0.001 0.001
- added link rear_right_axle_link, mass 0.23739; collision cylinder length=0.05 radius=0.05; visual mesh filename=package://swerve_description/meshes/SwerveAxle.stl scale=0.001 0.001 0.001
- added link rear_right_wheel_link, mass 0.23133211; collision cylinder length=0.0381 radius=0.0508; visual mesh filename=package://swerve_description/meshes/SwerveWheel.stl scale=0.001 0.001 0.001
Joints:
- removed joint back_left_axle_joint
- removed joint back_left_wheel_joint
- removed joint back_right_axle_joint
- removed joint back_right_wheel_joint
- added joint rear_left_axle_joint: type continuous, parent swerve_chassis_link, child rear_left_axle_link, origin xyz=0.301625 0.06905599999999999 -0.301625 rpy=1.5707963267948966 0 0, axis 0 0 1
- added joint rear_left_wheel_joint: type continuous, parent rear_left_axle_link, child rear_left_wheel_link, origin xyz=-0.022 0 0.065 rpy=0 0 0, axis 1 0 0
- added joint rear_right_axle_joint: type continuous, parent swerve_chassis_link, child rear_right_axle_link, origin xyz=-0.301625 0.06905599999999999 -0.301625 rpy=1.5707963267948966 0 0, axis 0 0 1
- added joint rear_right_wheel_joint: type continuous, parent rear_right_axle_link, child rear_right_wheel_link, origin xyz=-0.022 0 0.065 rpy=0 0 0, axis 1 0 0

Commit message: added field

File: src/swerve_description/swerve.urdf (robot description, URDF)
Before this commit: robot swerve, 10 links, 9 joints
Links:
- removed link rear_left_axle_link
- removed link rear_left_wheel_link
- removed link rear_right_axle_link
- removed link rear_right_wheel_link
- added link back_left_axle_link, mass 0.23739; collision cylinder length=0.05 radius=0.05; visual mesh filename=package://swerve_description/meshes/SwerveAxle.stl scale=0.001 0.001 0.001
- added link back_left_wheel_link, mass 0.23133211; collision cylinder length=0.0381 radius=0.0508; visual mesh filename=package://swerve_description/meshes/SwerveWheel.stl scale=0.001 0.001 0.001
- added link back_right_axle_link, mass 0.23739; collision cylinder length=0.05 radius=0.05; visual mesh filename=package://swerve_description/meshes/SwerveAxle.stl scale=0.001 0.001 0.001
- added link back_right_wheel_link, mass 0.23133211; collision cylinder length=0.0381 radius=0.0508; visual mesh filename=package://swerve_description/meshes/SwerveWheel.stl scale=0.001 0.001 0.001
Joints:
- removed joint rear_left_axle_joint
- removed joint rear_left_wheel_joint
- removed joint rear_right_axle_joint
- removed joint rear_right_wheel_joint
- added joint back_left_axle_joint: type continuous, parent swerve_chassis_link, child back_left_axle_link, origin xyz=0.301625 0.06905599999999999 -0.301625 rpy=1.5707963267948966 0 0, axis 0 0 1
- added joint back_left_wheel_joint: type continuous, parent back_left_axle_link, child back_left_wheel_link, origin xyz=-0.022 0 0.065 rpy=0 0 0, axis 1 0 0
- added joint back_right_axle_joint: type continuous, parent swerve_chassis_link, child back_right_axle_link, origin xyz=-0.301625 0.06905599999999999 -0.301625 rpy=1.5707963267948966 0 0, axis 0 0 1
- added joint back_right_wheel_joint: type continuous, parent back_right_axle_link, child back_right_wheel_link, origin xyz=-0.022 0 0.065 rpy=0 0 0, axis 1 0 0
